File: PhaethonBrdArduino/PhaetonArduinoBrd.sch (EAGLE design)
At the start: 43 parts, among them IC2 LM2596S, Q1 32.768 Hz, SW1 EC12E_SW

Commit message: New design, before Checks
Parts:
- removed ANALOG, J6: (no value), pinhead:PINHD-1X6
- removed C_INPUT: 330uF, resistor:CPOL-EU140CLH-1010
- removed C_OUTPUT: 3.3nF, resistor:CPOL-EU140CLH-1010
- removed D1: MBRS340T3, diode:MBRS340T3
- removed IC2: LM2596S, national-semiconductor:LM2596S
- removed J1, J2, J5, POWER: (no value), SmartPrj:PINHD-1X8TH
- removed J3, J4: (no value), SmartPrj:PINHD-1X10TH
- removed L1: 68uH, inductor-coilcraft:MSS1260
- removed RESET: (no value), switch-omron:10-XX
- added C10, C12: 1uF, resistor:C-EUC0402
- added C5, C9: 0.1uF, microbuilder:CAP_CERAMIC_0805MP
- added C6, C7: 3.3nF, rcl:C-EUC0504
- added C8: 100uF, rcl:CPOL-EUCT7343
- added CN1: (no value), microbuilder:USBMICRO_20329
- added C_INPUT1: 47uF, resistor:CPOL-EUC
- added D2: 3.6v, microbuilder:DIODESOD-323
- added D3, D5: SCHOTTKY, s1x_10:SCHOTTKY
- added D4: 3.6V, microbuilder:DIODESOD-323
- added IC1: ATmega328P, microbuilder:MEGA8-MI
- added LT1376-5: LE33, lt1376:LE33
- added OUTPUT2, U$3, U$5, U$6: MINICONECTOR, pcb_terminal:MINICONECTOR
- added Q2: reset, microbuilder:SWITCH_TACT_SMT4.6X2.8
- added Q3, Q4: BC847BS, transistor-small-signal:BC847BS
- added R14, R15: 68, resistor:R-EU_R0603
- added R16: 1.5K, resistor:R-EU_R0603
- added R17: 10K, resistor:R-EU_R0603
- added RN1, RN2: 10K, resistor-array:741-8_S
- added RN3: 100K, resistor-array:741-8_S
- added U$1: (no value), inductor-coilcraft:LPS3314-103MRB
- added Y1: 16MHz, SparkFun:RESONATORSMD
- C1, C3, C4: device rcl:C-EUC0805 -> rcl:C-EUC0504
- C2: device rcl:C-EUC0805K -> rcl:C-EUC0504
- G1: value BATTERY-HOLDER_11.6MM -> CR1216; device battery:BATTERY-HOLDER_11.6MM -> battery:CR1216
- R3, R4, R7: value 10K\ -> 100K
- R9: value 20K -> 100K
Connections:
- removed net +9V: J2.8, POWER.8
- removed net A0: ANALOG.1, J6.1, R11.2
- removed net A1: ANALOG.2, J6.2, R13.2
- removed net A2: ANALOG.3, J6.3, R12.2
- removed net N$222: J3.8, J4.8
- removed net N$223: J2.4, POWER.4
- removed net N$25: J2.6, POWER.6
- removed net N$31: J2.2, POWER.2
- removed net N$32: J2.1, POWER.1
- removed net N$97: DS1307.VBAT, G1.+
- removed net OUTPUT1: D1.C, IC2.OUT, L1.P$1
- removed net OUTPUT5V: C_OUTPUT.+, IC2.FB, L1.P$2, SJ1.1
- removed net PIN0: J1.1, J5.1
- removed net PIN1: J1.2, J5.2
- removed net PIN10: J3.3, J4.3
- removed net PIN7: DISPLAYCONNECTOR.3, J1.8, J5.8
- removed net PIN8: DISPLAYCONNECTOR.4, J3.1, J4.1
- removed net PIN9: J3.2, J4.2
- new net A6: IC1.ADC6
- new net AREF: C5.1, IC1.AREF
- new net BLUELED: IC1.PC0(ADC0), R11.2
- new net D+: CN1.D+, D2.C, R15.1
- new net D-: CN1.D-, D4.C, R14.1, R16.1
- new net D10: IC1.PB2(SS/OC1B), RN1D.1
- new net D7: IC1.PD7(AIN1), R14.2
- new net D8: IC1.PB0(ICP), RN1A.1
- new net D9: IC1.PB1(OC1A), RN2C.1
- new net DC/DC_OUTPUT: C8.+, D3.A, LT1376-5.BIAS, LT1376-5.FB/SENSE, SJ1.1, U$1.P$1
- new net GREENLED: IC1.PC2(ADC2), R13.2
- new net N$10: OUTPUT2.P$1, Q3A.C, RN3A.1
- new net N$11: C6.2, LT1376-5.VC
- new net N$12: C7.2, D3.C, LT1376-5.BOOST
- new net N$13: Q3B.C, RN3B.1, U$3.P$1
- new net N$14: C7.1, D5.C, LT1376-5.VSW, U$1.P$2
- new net N$15: Q4A.B, RN2A.1, RN2B.1
- new net N$16: Q3A.B, RN1A.2, RN1B.2
- new net N$17: Q3B.B, RN1C.1, RN1D.2
- new net N$18: Q4B.B, RN2C.2, RN2D.2
- new net N$19: Q4B.C, RN3D.1, U$6.P$1
- new net N$20: Q4A.C, RN3C.2, U$5.P$1
- new net N$7: IC1.PB7(XTAL2/TOSC2), Y1.3
- new net N$8: IC1.PB6(XTAL1/TOSC1), Y1.1
- new net REDLED: IC1.PC1(ADC1), R12.2
- new net RXD: IC1.PD0(RXD), RN2B.2
- new net TXD: IC1.PD1(TXD)
- new net VBAT: DS1307.VBAT, G1.+, IC1.ADC7
- new net VBUS: CN1.VBUS
- net +24V: now also C10.2, C12.2, C_INPUT1.+, LT1376-5.VIN, RN3A.2, RN3B.2, RN3C.1, RN3D.2; no longer C_INPUT.+, IC2.VIN
- net +5V: now also C9.2, DISPLAYCONNECTOR.2, IC1.AVCC, IC1.VCC@1, IC1.VCC@2, R16.2, R17.2; no longer DISPLAYCONNECTOR.1, J2.5, POWER.5
- net A3: now also IC1.PC3(ADC3); no longer ANALOG.4, J6.4
- net GND: now also C10.1, C12.1, C5.2, C6.1, C8.-, C9.1, CN1.GND, C_INPUT1.-, D2.A, D4.A, D5.A, DISPLAYCONNECTOR.1, IC1.GND, IC1.GND@1, IC1.GND@2, IC1.THERMAL, LT1376-5.GND, Q2.S, Q2.S1, Q3A.E, Q3B.E, Q4A.E, Q4B.E, RN1B.1, RN1C.2, RN2A.2, RN2D.1, Y1.2; no longer C_INPUT.-, C_OUTPUT.-, D1.A, DISPLAYCONNECTOR.2, IC2.!ON!/OFF, IC2.GND, J2.7, J3.7, J4.7, POWER.7, RESET.S, RESET.S1
- net MISO: now also IC1.PB4(MISO); no longer J3.5, J4.5
- net MOSI: now also IC1.PB3(MOSI/OC2); no longer J3.4, J4.4
- net PIN2: now also IC1.PD2(INT0), R15.2; no longer J1.3, J5.3
- net PIN3: now also IC1.PD3(INT1); no longer J1.4, J5.4
- net PIN4: now also IC1.PD4(XCK/T0); no longer J1.5, J5.5
- net PIN5: now also IC1.PD5(T1); no longer J1.6, J5.6
- net PIN6: now also IC1.PD6(AIN0); no longer J1.7, J5.7
- net RESET: now also IC1.PC6(/RESET), Q2.P, Q2.P1, R17.1; no longer J2.3, POWER.3, RESET.P, RESET.P1
- net SCK: now also IC1.PB5(SCK); no longer J3.6, J4.6
- net SCL: now also DISPLAYCONNECTOR.4, IC1.PC5(ADC5/SCL); no longer ANALOG.6, J3.10, J4.10, J6.6
- net SDA: now also DISPLAYCONNECTOR.3, IC1.PC4(ADC4/SDA); no longer ANALOG.5, J3.9, J4.9, J6.5
Other:
- note added: "OLED disp con."
- note added: "dc/dc 25V / 5V"
- note removed: "TM1637 con."
- note removed: "dc/dc 40V / 5V"
- moved on the sheet: G1, ICSP, SJ1
