File: PhaethonBrdArduino/PhaetonArduinoBrd.sch (EAGLE design)
At the start: 60 parts, among them IC1 ATmega328P, Q1 32.768 Hz, Q2 reset, Q3 BC847BS, Q4 BC847BS, SW1 EC12E_SW, Y1 16MHz

Commit message: Phaethon V2 in Seedstudio
Parts:
- removed C_INPUT1: 47uF, resistor:CPOL-EUC
- removed U$1: (no value), inductor-coilcraft:LPS3314-103MRB
- added C11: 33uF, Eagle_CAPACITORS:WCAP-ASLI_5X5.5(DXL)
- added U$4: 10uH\, inductor-coilcraft3:LPS3314-103MRB
- C7: value 3.3nF -> 0.1uF
- CN1: device microbuilder:USBMICRO_20329 -> microbuilder:USBMINIB
- renumbered DISPLAYCONNECTOR to OLED
Connections:
- net +24V: now also C11.1; no longer C_INPUT1.+
- net DC/DC_OUTPUT: now also U$4.P$2; no longer U$1.P$1
- net GND: now also C11.2; no longer C_INPUT1.-
- net N$14: now also U$4.P$1; no longer U$1.P$2
Changed lines of the file:
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@@
 <part name="SV1" library="con-amp-mt6" deviceset="MT6-3" device=""/>
 <part name="R11" library="SparkFun" deviceset="RESISTOR" device="" value="125"/>
-<part name="DISPLAYCONNECTOR" library="con-amp-quick" deviceset="M04" device=""/>
+<part name="OLED" library="con-amp-quick" deviceset="M04" device=""/>
 <part name="GND18" library="supply1" deviceset="GND" device=""/>
 <part name="GND19" library="supply1" deviceset="GND" device=""/>
@@
 <part name="GND17" library="supply1" deviceset="GND" device=""/>
 <part name="R16" library="resistor" deviceset="R-EU_" device="R0603" value="1.5K"/>
-<part name="CN1" library="microbuilder" deviceset="USB" device="MICRO_20329"/>
+<part name="CN1" library="microbuilder" deviceset="USB" device="MINIB"/>
 <part name="U$2" library="microbuilder" deviceset="VBUS" device=""/>
 <part name="D2" library="microbuilder" deviceset="DIODE" device="SOD-323" value="3.6v"/>
@@
 <part name="D3" library="s1x_10" deviceset="SCHOTTKY" device=""/>
 <part name="D5" library="s1x_10" deviceset="SCHOTTKY" device=""/>
-<part name="C_INPUT1" library="resistor" deviceset="CPOL-EU" device="C" value="47uF"/>
 <part name="P+18" library="supply1" deviceset="+24V" device=""/>
 <part name="GND1" library="supply1" deviceset="GND" device=""/>
@@
 <part name="C6" library="rcl" deviceset="C-EU" device="C0504" value="3.3nF"/>
 <part name="GND14" library="supply1" deviceset="GND" device=""/>
-<part name="C7" library="rcl" deviceset="C-EU" device="C0504" value="3.3nF"/>
+<part name="C7" library="rcl" deviceset="C-EU" device="C0504" value="0.1uF"/>
 <part name="GND15" library="supply1" deviceset="GND" device=""/>
 <part name="C8" library="rcl" deviceset="CPOL-EU" device="CT7343" value="100uF"/>
 <part name="GND16" library="supply1" deviceset="GND" device=""/>
-<part name="U$1" library="inductor-coilcraft" deviceset="LPS3314-103MRB" device=""/>
 <part name="C9" library="microbuilder" deviceset="CAP_CERAMIC" device="_0805MP" value="0.1uF"/>
 <part name="GND13" library="supply1" deviceset="GND" device=""/>
@@
 <part name="U$5" library="pcb_terminal" deviceset="MINICONECTOR" device=""/>
 <part name="U$6" library="pcb_terminal" deviceset="MINICONECTOR" device=""/>
+<part name="U$4" library="inductor-coilcraft3" deviceset="LPS3314-103MRB" device="" value="10uH\"/>
+<part name="C11" library="Eagle_CAPACITORS" deviceset="WCAP-ASLI" device="_5X5.5(DXL)" value="33uF"/>
 </parts>
 <sheets>
@@
 <instance part="SV1" gate="-3" x="144.78" y="-12.7" rot="R270"/>
 <instance part="R11" gate="G$1" x="78.74" y="93.98" rot="R270"/>
-<instance part="DISPLAYCONNECTOR" gate="G$1" x="195.58" y="-15.24" rot="R270"/>
+<instance part="OLED" gate="G$1" x="195.58" y="-15.24" rot="R270"/>
 <instance part="GND18" gate="1" x="203.2" y="93.98" rot="R90"/>
 <instance part="GND19" gate="1" x="203.2" y="86.36" rot="R90"/>
@@
 <attribute name="NAME" x="63.0174" y="-27.94" size="1.778" layer="95" rot="R90"/>
 </instance>
-<instance part="C_INPUT1" gate="G$1" x="43.18" y="-17.78" smashed="yes">
-<attribute name="NAME" x="40.1574" y="-24.257" size="1.778" layer="95" rot="R90"/>
-<attribute name="VALUE" x="47.7774" y="-24.257" size="1.778" layer="96" rot="R90"/>
-</instance>
 <instance part="P+18" gate="1" x="43.18" y="-2.54"/>
 <instance part="GND1" gate="1" x="43.18" y="-33.02"/>
@@
 </instance>
 <instance part="GND16" gate="1" x="60.96" y="2.54" rot="R180"/>
-<instance part="U$1" gate="G$1" x="78.74" y="-30.48" rot="R270"/>
 <instance part="C9" gate="G$1" x="312.42" y="-76.2" rot="R180"/>
 <instance part="GND13" gate="1" x="312.42" y="-83.82"/>
@@
 <instance part="U$5" gate="G$1" x="378.46" y="7.62" rot="R90"/>
 <instance part="U$6" gate="G$1" x="358.14" y="22.86" rot="R270"/>
+<instance part="U$4" gate="G$1" x="78.74" y="-30.48" rot="R90"/>
+<instance part="C11" gate="G$1" x="43.18" y="-20.32"/>
 </instances>
 <busses>
@@
 </segment>
 <segment>
-<pinref part="DISPLAYCONNECTOR" gate="G$1" pin="2"/>
+<pinref part="OLED" gate="G$1" pin="2"/>
 <wire x1="195.58" y1="-20.32" x2="195.58" y2="-25.4" width="0.1524" layer="91"/>
 <label x="195.58" y="-27.94" size="1.778" layer="95" rot="R90"/>
@@
 </segment>
 <segment>
-<pinref part="DISPLAYCONNECTOR" gate="G$1" pin="1"/>
+<pinref part="OLED" gate="G$1" pin="1"/>
 <wire x1="193.04" y1="-20.32" x2="193.04" y2="-25.4" width="0.1524" layer="91"/>
 <label x="193.04" y="-25.4" size="1.778" layer="95" rot="R90"/>
-</segment>
-<segment>
-<pinref part="C_INPUT1" gate="G$1" pin="-"/>
-<pinref part="GND1" gate="1" pin="GND"/>
-<wire x1="43.18" y1="-30.48" x2="43.18" y2="-22.86" width="0.1524" layer="91"/>
 </segment>
 <segment>
@@
 <pinref part="RN2" gate="A" pin="2"/>
 </segment>
+<segment>
+<pinref part="GND1" gate="1" pin="GND"/>
+<pinref part="C11" gate="G$1" pin="2"/>
+<wire x1="43.18" y1="-30.48" x2="43.18" y2="-22.86" width="0.1524" layer="91"/>
+</segment>
 </net>
 <net name="RESET" class="0">
@@
 </segment>
 <segment>
-<pinref part="DISPLAYCONNECTOR" gate="G$1" pin="3"/>
+<pinref part="OLED" gate="G$1" pin="3"/>
 <wire x1="198.12" y1="-20.32" x2="198.12" y2="-27.94" width="0.1524" layer="91"/>
 <label x="198.12" y="-30.48" size="1.778" layer="95" rot="R90"/>
@@
 </segment>
 <segment>
-<pinref part="DISPLAYCONNECTOR" gate="G$1" pin="4"/>
+<pinref part="OLED" gate="G$1" pin="4"/>
 <wire x1="200.66" y1="-20.32" x2="200.66" y2="-27.94" width="0.1524" layer="91"/>
 <label x="200.66" y="-33.02" size="1.778" layer="95" rot="R90"/>
@@
 <wire x1="154.94" y1="91.44" x2="162.56" y2="91.44" width="0.1524" layer="91"/>
 <label x="157.48" y="91.44" size="1.778" layer="95"/>
+<junction x="154.94" y="91.44"/>
 </segment>
 <segment>
@@
 <wire x1="167.64" y1="99.06" x2="160.02" y2="99.06" width="0.1524" layer="91"/>
 <label x="160.02" y="99.06" size="1.778" layer="95"/>
+<junction x="167.64" y="99.06"/>
 </segment>
 <segment>
@@
 <wire x1="152.4" y1="-38.1" x2="154.94" y2="-38.1" width="0.1524" layer="91"/>
 <label x="152.4" y="-38.1" size="1.778" layer="95"/>
-</segment>
-<segment>
-<pinref part="C_INPUT1" gate="G$1" pin="+"/>
-<pinref part="P+18" gate="1" pin="+24V"/>
-<wire x1="43.18" y1="-5.08" x2="43.18" y2="-15.24" width="0.1524" layer="91"/>
 </segment>
 <segment>
@@
 <pinref part="RN3" gate="C" pin="1"/>
 </segment>
+<segment>
+<pinref part="C11" gate="G$1" pin="1"/>
+<pinref part="P+18" gate="1" pin="+24V"/>
+<wire x1="43.18" y1="-15.24" x2="43.18" y2="-5.08" width="0.1524" layer="91"/>
+</segment>
 </net>
 <net name="OUTPUT" class="0">
@@
 <label x="53.34" y="-10.16" size="1.778" layer="95" rot="R90"/>
 <pinref part="C8" gate="G$1" pin="+"/>
+<junction x="53.34" y="-12.7"/>
 </segment>
 <segment>
@@
 </segment>
 <segment>
-<pinref part="U$1" gate="G$1" pin="P$1"/>
 <pinref part="LT1376-5" gate="G$1" pin="FB/SENSE"/>
 <wire x1="86.36" y1="-30.48" x2="91.44" y2="-30.48" width="0.1524" layer="91"/>
 <wire x1="91.44" y1="-30.48" x2="91.44" y2="-20.32" width="0.1524" layer="91"/>
 <label x="91.44" y="-25.4" size="1.778" layer="95"/>
+<pinref part="U$4" gate="G$1" pin="P$2"/>
 </segment>
 </net>
@@
 <wire x1="66.04" y1="-17.78" x2="68.58" y2="-17.78" width="0.1524" layer="91"/>
 <junction x="63.5" y="-20.32"/>
-<pinref part="U$1" gate="G$1" pin="P$2"/>
 <wire x1="71.12" y1="-30.48" x2="71.12" y2="-25.4" width="0.1524" layer="91"/>
 <wire x1="71.12" y1="-25.4" x2="63.5" y2="-25.4" width="0.1524" layer="91"/>
 <junction x="63.5" y="-25.4"/>
+<pinref part="U$4" gate="G$1" pin="P$1"/>
 </segment>
 </net>
@@
 </sheet>
 </sheets>
+<errors>
+</errors>
 </schematic>
 </drawing>
