File: PhaethonBrdArduino/PhaetonArduinoBrd.brd (EAGLE design)
At the start: 68.6 x 53.3 mm, 43 parts, among them IC2 LM2596S, Q1 32.768 Hz, SW1 EC12E_SW

Commit message: New design, before Checks
Parts:
- removed ANALOG, J6: (no value), pinhead:1X06
- removed C_INPUT: 330uF, resistor:140CLH-1010
- removed C_OUTPUT: 3.3nF, resistor:140CLH-1010
- removed D1: MBRS340T3, diode:SMC
- removed IC2: LM2596S, national-semiconductor:TO263-5
- removed J1, J2, J5, POWER: (no value), SmartPrj:1X08-TH
- removed J3, J4: (no value), SmartPrj:1X10-TH
- removed L1: 68uH, inductor-coilcraft:MSS1260
- removed RESET: (no value), switch-omron:B3F-10XX
- added C10, C12: 1uF, resistor:C0402
- added C5, C9: 0.1uF, microbuilder:_0805MP
- added C6, C7: 3.3nF, rcl:C0504
- added C8: 100uF, rcl:CT7343
- added CN1: (no value), microbuilder:4UCONN_20329
- added C_INPUT1: 47uF, resistor:PANASONIC_C
- added D2: 3.6v, microbuilder:SOD-323
- added D3, D5: SCHOTTKY, s1x_10:DO214
- added D4: 3.6V, microbuilder:SOD-323
- added IC1: ATmega328P, microbuilder:MLF32-TH
- added LT1376-5: LE33, lt1376:SO08
- added OUTPUT2, U$3, U$5, U$6: MINICONECTOR, pcb_terminal:SMD
- added Q2: reset, microbuilder:BTN_KMR2_4.6X2.8
- added Q3, Q4: BC847BS, transistor-small-signal:SOT363_PHILIPS
- added R14, R15: 68, resistor:R0603
- added R16: 1.5K, resistor:R0603
- added R17: 10K, resistor:R0603
- added RN1, RN2: 10K, resistor-array:741-8
- added RN3: 100K, resistor-array:741-8
- added U$1: (no value), inductor-coilcraft:103MRB
- added Y1: 16MHz, SparkFun:RESONATOR-SMD
- C1, C3, C4: device rcl:C0805 -> rcl:C0504
- C2: device rcl:C0805K -> rcl:C0504
- G1: value BATTERY-HOLDER_11.6MM -> CR1216; device battery:CELL_RETAINER_11.6MM -> battery:SMTU1225-LF
- R3, R4, R7: value 10K\ -> 100K
- R9: value 20K -> 100K
- moved R1 41.6 mm to (13.1, 41.2)
- moved C2 33.5 mm to (39.3, 18.8), turned to 0 degrees
- moved R2 33.4 mm to (12.6, 30.1), turned to 0 degrees
- moved DS1307 32.7 mm to (14.1, 35.4)
- moved Q1 31.5 mm to (21.2, 34.6)
- moved ICSP 30.1 mm to (40.8, 9.91), turned to 180 degrees
- moved R5 28.3 mm to (34.2, 36.8), turned to 90 degrees
- moved ADT 28.2 mm to (39.3, 23.4)
- moved R6 26.7 mm to (29.2, 36.7), turned to 90 degrees
- moved R7 25.8 mm to (31.8, 36.8), turned to 270 degrees
- moved LED 24.2 mm to (19.8, 40.4)
- moved C4 23.3 mm to (31.9, 32.3)
- moved C1 22.5 mm to (27.7, 32.5)
- moved R4 21.4 mm to (30.7, 41.5)
- moved SW1 21.2 mm to (31.9, 37.4)
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Connections:
- removed net +9V: J2.8, POWER.8
- removed net A0: ANALOG.1, J6.1, R11.2
- removed net A1: ANALOG.2, J6.2, R13.2
- removed net A2: ANALOG.3, J6.3, R12.2
- removed net N$222: J3.8, J4.8
- removed net N$223: J2.4, POWER.4
- removed net N$25: J2.6, POWER.6
- removed net N$31: J2.2, POWER.2
- removed net N$32: J2.1, POWER.1
- removed net N$97: DS1307.3, G1.P+@1, G1.P+@2
- removed net OUTPUT1: D1.C, IC2.2, L1.P$1
- removed net OUTPUT5V: C_OUTPUT.+, IC2.4, L1.P$2, SJ1.1
- removed net PIN0: J1.1, J5.1
- removed net PIN1: J1.2, J5.2
- removed net PIN10: J3.3, J4.3
- removed net PIN7: DISPLAYCONNECTOR.3, J1.8, J5.8
- removed net PIN8: DISPLAYCONNECTOR.4, J3.1, J4.1
- removed net PIN9: J3.2, J4.2
- new net A6: IC1.19
- new net AREF: C5.1, IC1.20
- new net BLUELED: IC1.23, R11.2
- new net D+: CN1.D+, D2.C, R15.1
- new net D-: CN1.D-, D4.C, R14.1, R16.1
- new net D10: IC1.14, RN1.4
- new net D7: IC1.11, R14.2
- new net D8: IC1.12, RN1.1
- new net D9: IC1.13, RN2.3
- new net DC/DC_OUTPUT: C8.+, D3.A, LT1376-5.4, LT1376-5.7, SJ1.1, U$1.1
- new net GREENLED: IC1.25, R13.2
- new net N$10: OUTPUT2.1, Q3.6, RN3.1
- new net N$11: C6.2, LT1376-5.8
- new net N$12: C7.2, D3.C, LT1376-5.1
- new net N$13: Q3.3, RN3.2, U$3.1
- new net N$14: C7.1, D5.C, LT1376-5.3, U$1.2
- new net N$15: Q4.2, RN2.1, RN2.2
- new net N$16: Q3.2, RN1.7, RN1.8
- new net N$17: Q3.5, RN1.3, RN1.5
- new net N$18: Q4.5, RN2.5, RN2.6
- new net N$19: Q4.3, RN3.4, U$6.1
- new net N$20: Q4.6, RN3.6, U$5.1
- new net N$7: IC1.8, Y1.3
- new net N$8: IC1.7, Y1.1
- new net REDLED: IC1.24, R12.2
- new net RXD: IC1.30, RN2.7
- new net SHDN: LT1376-5.5
- new net TXD: IC1.31
- new net VBAT: DS1307.3, G1.P+, IC1.22
- new net VBUS: CN1.VBUS
- net +24V: now also C10.2, C12.2, C_INPUT1.+, LT1376-5.2, RN3.3, RN3.5, RN3.7, RN3.8; no longer C_INPUT.+, IC2.1
- net +5V: now also C9.2, DISPLAYCONNECTOR.2, IC1.18, IC1.4, IC1.6, R16.2, R17.2; no longer DISPLAYCONNECTOR.1, J2.5, POWER.5
- net A3: now also IC1.26; no longer ANALOG.4, J6.4
- net GND: now also C10.1, C12.1, C5.2, C6.1, C8.-, C9.1, CN1.BASE@1, CN1.BASE@2, CN1.GND, CN1.SPRT@1, CN1.SPRT@2, CN1.SPRT@3, CN1.SPRT@4, C_INPUT1.-, D2.A, D4.A, D5.A, DISPLAYCONNECTOR.1, G1.P-, IC1.21, IC1.3, IC1.5, IC1.TH, LT1376-5.6, Q2.B, Q2.B', Q3.1, Q3.4, Q4.1, Q4.4, RN1.2, RN1.6, RN2.4, RN2.8, Y1.2; no longer C_INPUT.-, C_OUTPUT.-, D1.A, DISPLAYCONNECTOR.2, G1.N-, IC2.3, IC2.5, J2.7, J3.7, J4.7, POWER.7, RESET.1, RESET.2
- net MISO: now also IC1.16; no longer J3.5, J4.5
- net MOSI: now also IC1.15; no longer J3.4, J4.4
- net PIN2: now also IC1.32, R15.2; no longer J1.3, J5.3
- net PIN3: now also IC1.1; no longer J1.4, J5.4
- net PIN4: now also IC1.2; no longer J1.5, J5.5
- net PIN5: now also IC1.9; no longer J1.6, J5.6
- net PIN6: now also IC1.10; no longer J1.7, J5.7
- net RESET: now also IC1.29, Q2.A, Q2.A', R17.1; no longer J2.3, POWER.3, RESET.3, RESET.4
- net SCK: now also IC1.17; no longer J3.6, J4.6
- net SCL: now also DISPLAYCONNECTOR.4, IC1.28; no longer ANALOG.6, J3.10, J4.10, J6.6
- net SDA: now also DISPLAYCONNECTOR.3, IC1.27; no longer ANALOG.5, J3.9, J4.9, J6.5
Routing:
- net GND: track 243.5 -> 160.9 mm, vias 1 -> 32
- net D10: track 0.00 -> 74.3 mm, vias 0 -> 4
- net A2: track 71.4 -> 0.00 mm, vias 1 -> 0
- net +24V: track 38.5 -> 108.7 mm, vias 4 -> 2
- net VBAT: track 0.00 -> 55.5 mm, vias 0 -> 3
- net RESET: track 124.9 -> 76.1 mm, vias 7 -> 1
- net A0: track 48.5 -> 0.00 mm, vias 1 -> 0
- net D9: track 0.00 -> 47.4 mm, vias 0 -> 2
- net D7: track 0.00 -> 47.4 mm, vias 0 -> 2
- net A1: track 45.3 -> 0.00 mm, vias 3 -> 0
- net D8: track 0.00 -> 42.2 mm, vias 0 -> 4
- net OUTPUT5V: track 40.8 -> 0.00 mm
- net BLUELED: track 0.00 -> 39.6 mm, vias 0 -> 2
- net PIN7: track 39.5 -> 0.00 mm
- net PIN8: track 38.9 -> 0.00 mm
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- added copper zone on layer 1, net N$23
- added copper zone on layer 16, net N$23
- removed copper zone on layer 1, net OUTPUT1
- removed copper zone on layer 1, net OUTPUT5V
Other:
- board size 68.6 x 53.3 mm -> 58 x 50 mm
- board text added: "G"
- board text added: "W/W1"
- board text added: "W2"
- board text added: "Y/Y1"
- board text added: "Y2"
- board text removed: "0"
- board text removed: "0 1 2 3 4 5"
- board text removed: "10"
- board text removed: "11"
- board text removed: "12"
- board text removed: "13"
- board text removed: "3"
- board text removed: "3.3V"
- board text removed: "3V3"
- board text removed: "4"
- board text removed: "5"
- board text removed: "5V"
- board text removed: "5V Gnd 9V"
- board text removed: "6"
- board text removed: "7"
- board text removed: "8"
- board text removed: "9"
- board text removed: "ANALOG"
- board text removed: "AREF"
- board text removed: "DIGITAL"
- board text removed: "ETH"
- board text removed: "GND"
- board text removed: "IOREF"
- board text removed: "RES"
- board text removed: "RST"
- board text removed: "SCL"
- board text removed: "SDA"
- board text removed: "USB"
- board text removed: "VIN"

Commit message: Phaethon V2 in Seedstudio
Parts:
- removed C_INPUT1: 47uF, resistor:PANASONIC_C
- removed U$1: (no value), inductor-coilcraft:103MRB
- added C11: 33uF, Eagle_CAPACITORS:3X1.6X1.4(BXCXA)
- added U$4: 10uH\, inductor-coilcraft3:103MRB
- C7: value 3.3nF -> 0.1uF
- CN1: device microbuilder:4UCONN_20329 -> microbuilder:USB-MINIB
- moved R9 6.65 mm to (7.62, 47.4)
- moved R15 6.25 mm to (45.2, 21.1), turned to 180 degrees
- moved C10 5.93 mm to (2.79, 43.1)
- moved R14 5.60 mm to (45.2, 18.0), turned to 0 degrees
- moved R16 2.53 mm to (47.2, 23.4)
- moved R7 0.25 mm to (31.5, 36.8)
- moved OUTPUT2 0.16 mm to (53.3, 37.0)
- moved U$3 0.16 mm to (53.3, 41.0)
- moved U$5 0.16 mm to (53.3, 33.0)
- moved U$6 0.16 mm to (53.3, 29.0)
- moved C4 0.13 mm to (32.1, 32.3)
- renumbered DISPLAYCONNECTOR to OLED
Connections:
- net +24V: now also C11.1; no longer C_INPUT1.+
- net DC/DC_OUTPUT: now also U$4.2; no longer U$1.1
- net GND: now also C11.2; no longer CN1.BASE@1, CN1.BASE@2, CN1.SPRT@1, CN1.SPRT@2, CN1.SPRT@3, CN1.SPRT@4, C_INPUT1.-
- net N$14: now also U$4.1; no longer U$1.2
Routing:
- net GND: track 160.9 -> 96.2 mm, vias 32 -> 18
- net D+: track 19.5 -> 9.04 mm
- net +24V: track 108.7 -> 118.4 mm, vias 2 -> 5
- net D8: track 42.2 -> 50.3 mm, vias 4 -> 8
- net D-: track 13.8 -> 19.7 mm, vias 1 -> 2
- net OUTPUT: track 11.4 -> 16.9 mm
- net N$17: track 9.79 -> 4.72 mm
- net PIN2: track 50.2 -> 47.6 mm, vias 5 -> 7
- net N$16: track 4.95 -> 7.44 mm
- net +5V: track 174.4 -> 176.1 mm
- net N$14: track 22.5 -> 24.0 mm
- net N$15: track 7.93 -> 6.75 mm
- net PIN6: track 24.3 -> 23.4 mm
- net MOSI: track 53.2 -> 52.5 mm
- net SCL: track 68.5 -> 69.2 mm
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Other:
- board text added: "+"
